Commit message: attempt

File: ws_rviz/src/urdf02_gazebo/urdf/car.xacro (robot description, xacro)
@@ -5,3 +5,8 @@
     <xacro:include filename="demo02_camera.xacro" />
     <xacro:include filename="demo02_laser.xacro" />
+    <xacro:include filename="rmus_map_2.urdf" />
+    <xacro:include filename="gazebo/move.xacro" />
+    <xacro:include filename="gazebo/laser.xacro" />
+    <xacro:include filename="gazebo/camera.xacro" />
+    <xacro:include filename="gazebo/kinetic.xacro" />
 </robot>

File: ws_rviz/src/urdf02_gazebo/urdf/rmus_map_2.urdf (robot description, URDF)
Before this commit: robot rmus_map_2, 1 links, 0 joints
Links:
- link base_link: geometry collision mesh filename=package://meshes/base_link.stl; visual mesh filename=package://meshes/base_link.stl
