Commit message: Turn the repo into a runnable ROS Noetic showcase
- Vendor the racecar packages in place of the dangling submodule links and port
  them to Noetic: OpenCV 4 build fixes, Python 3 nodes, gmapping frames that
  match the simulation, repeated goals in path_pursuit.py.
- Add a Docker image that builds both workspaces and runs Gazebo and RViz
  headlessly, with a noVNC browser desktop, demo recording and an end-to-end
  navigation test that CI runs on every push.
- Add one-command launch files for the navigation and mapping demos.
- Fix absolute mesh paths in the RMUS world, drop IDE folders and the broken
  terminal wrapper scripts.
- Rewrite the README around the recorded demos; add MIT license.

File: ws_rviz/src/urdf02_gazebo/urdf/rmus_map_2.urdf (robot description, URDF)
Before this commit: robot rmus_map_2, 1 links, 0 joints
Links:
- link base_link: geometry collision mesh filename=package://rmus_map/meshes/base_link.stl; visual mesh filename=package://rmus_map/meshes/base_link.stl
